Commit message: fix: rewrite robot URDF with separate coloured links (no external meshes)
Root cause of invisible robot: package://warehouse_description/meshes/*.stl
paths are silently skipped by Gazebo when the package install directory has
not been updated. Only primitive geometry (the caster spheres) rendered.

Fix: eliminate ALL external file dependencies. Each coloured robot zone is
now a separate fixed-joint URDF link with its own <gazebo reference> material
block. Gazebo Classic colours each link independently — this is guaranteed
to work with no build-artifact dependencies.

Links and colours:
  base_link          — orange body box (0.9×0.65×0.4 m) + collision + inertia
  lid_link           — charcoal overhanging lid plate
  bumper_front_link  — charcoal front safety bar + yellow warning stripe
  bumper_rear_link   — charcoal rear safety bar
  accent_left/right  — charcoal side panels
  mast_link          — orange tapered two-cylinder identification mast
  sensor_ring_link   — dark-grey 360° LiDAR housing disc
  beacon_link        — bright blue safety beacon cylinder
  dome_link          — bright blue safety dome sphere  (~1.56 m above ground)
  wheel_left/right   — Gazebo/FlatBlack large drive wheels (r=0.170 m)
  caster_front/rear  — Gazebo/DarkGrey caster balls

Physics unchanged: mass=60 kg, wheel_radius=0.170 m, separation=0.580 m,
max_wheel_torque=80 Nm, max_wheel_acceleration=40 rad/s², spawn z=0.175 m.

Co-Authored-By: Claude Sonnet 4.6 <noreply@anthropic.com>
Claude-Session: https://claude.ai/code/session_016EwupYKQVrfCeF8yG8S6Li

File: src/warehouse_description/urdf/warehouse_robot.urdf.xacro (robot description, xacro)
@@ -1,5 +1,5 @@
 <?xml version="1.0"?>
 <robot name="warehouse_robot" xmlns:xacro="http://www.ros.org/wiki/xacro">
-  <!-- Args — kept identical for full launch-file compatibility -->
+  <!-- Args — identical to original for launch-file compatibility -->
   <xacro:arg name="robot_name"    default="robot1"/>
   <xacro:arg name="robot_id"      default="Robot_1"/>
@@ -9,19 +9,47 @@
   <xacro:property name="robot_ns" value="$(arg robot_name)"/>
   <!-- ═══════════════════════════════════════════════════════════════════
-       PHYSICS (spawn height z=0.175 = wheel_radius 0.170 + offset 0.005)
-       All visuals use package://warehouse_description/meshes/*.stl
-       which are installed by CMakeLists to share/warehouse_description/meshes/
+       PHYSICS  — spawn height z = 0.175 m  (= wheel_radius + |offset|)
+       Ground plane is at base_link z = −0.175 m
        ═══════════════════════════════════════════════════════════════════ -->
   <xacro:property name="base_mass"       value="60.0"/>
   <xacro:property name="wheel_radius"    value="0.170"/>
   <xacro:property name="wheel_width"     value="0.080"/>
-  <xacro:property name="wheel_sep_half"  value="0.290"/>
+  <xacro:property name="wheel_sep_half"  value="0.290"/>   <!-- 0.580 m axle / 2 -->
   <xacro:property name="wheel_offset_z"  value="-0.005"/>
   <xacro:property name="caster_radius"   value="0.050"/>
+  <!-- caster bottom must touch ground: caster_z = caster_radius − spawn_z = 0.050−0.175 -->
   <xacro:property name="caster_z"        value="-0.125"/>
-  <xacro:property name="caster_front_x"  value=" 0.390"/>
-  <xacro:property name="caster_rear_x"   value="-0.390"/>
-  <xacro:property name="body_z"          value="0.045"/>
-  <xacro:property name="body_h"          value="0.400"/>
+  <xacro:property name="caster_front_x"  value=" 0.395"/>
+  <xacro:property name="caster_rear_x"   value="-0.395"/>
+  <!-- Pre-computed geometry constants (base_link frame) -->
+  <!-- body_bottom = -0.175 + 0.020(clearance) = -0.155                  -->
+  <!-- body_z      = -0.155 + 0.200             =  0.045  (body centre)   -->
+  <!-- body_top    =  0.045 + 0.200             =  0.245                  -->
+  <!-- lid_cz      =  0.245 + 0.013             =  0.258                  -->
+  <!-- bumper_cz   = -0.155 + 0.130             = -0.025                  -->
+  <!-- mast_cz     =  0.271 + 0.450             =  0.721  (mast centre)   -->
+  <!-- beacon_cz   =  1.171 + 0.110             =  1.281                  -->
+  <!-- dome_cz     =  1.281 + 0.100 + 0.090     =  1.471                  -->
+  <xacro:property name="body_z"   value=" 0.045"/>
+  <xacro:property name="body_h"   value=" 0.400"/>
+  <!-- ════════════════════════════════════════
+       Helper macro: inertia-free visual link
+       (used for all decoration-only links)
+       ════════════════════════════════════════ -->
+  <xacro:macro name="visual_link" params="name">
+    <link name="${robot_ns}/${name}">
+      <inertial>
+        <mass value="0.001"/>
+        <inertia ixx="1e-9" iyy="1e-9" izz="1e-9" ixy="0" ixz="0" iyz="0"/>
+      </inertial>
+    </link>
+  </xacro:macro>
+  <xacro:macro name="fixed_joint" params="name parent child ox oy oz">
+    <joint name="${robot_ns}/${name}" type="fixed">
+      <parent link="${robot_ns}/${parent}"/>
+      <child  link="${robot_ns}/${child}"/>
+      <origin xyz="${ox} ${oy} ${oz}" rpy="0 0 0"/>
+    </joint>
+  </xacro:macro>
   <!-- ── base footprint ── -->
   <link name="${robot_ns}/base_footprint"/>
@@ -32,87 +60,220 @@
   </joint>
   <!-- ═══════════════════════════════════════════════════════════════════
-       BASE LINK — mesh-based industrial warehouse AMR
-       Each visual uses a separate STL so Gazebo can colour them
-       independently via material overrides.
+       1. BASE LINK — orange body box + collision + inertia
        ═══════════════════════════════════════════════════════════════════ -->
   <link name="${robot_ns}/base_link">
-    <!-- ── Main orange body ── -->
-    <visual name="body">
-      <origin xyz="0 0 0" rpy="0 0 0"/>
-      <geometry>
-        <mesh filename="package://warehouse_description/meshes/amr_body.stl"/>
-      </geometry>
-      <material name="amr_orange"><color rgba="1.00 0.55 0.00 1.0"/></material>
-    </visual>
-    <!-- ── Dark lid plate ── -->
-    <visual name="lid">
-      <origin xyz="0 0 0" rpy="0 0 0"/>
-      <geometry>
-        <mesh filename="package://warehouse_description/meshes/amr_lid.stl"/>
-      </geometry>
-      <material name="amr_charcoal"><color rgba="0.14 0.14 0.14 1.0"/></material>
-    </visual>
-    <!-- ── Front bumper ── -->
-    <visual name="bumper_front">
-      <origin xyz="0.480 0 0" rpy="0 0 0"/>
-      <geometry>
-        <mesh filename="package://warehouse_description/meshes/amr_bumper_front.stl"/>
-      </geometry>
-      <material name="amr_charcoal"/>
-    </visual>
-    <!-- ── Rear bumper ── -->
-    <visual name="bumper_rear">
-      <origin xyz="-0.480 0 0" rpy="0 0 0"/>
-      <geometry>
-        <mesh filename="package://warehouse_description/meshes/amr_bumper_rear.stl"/>
-      </geometry>
-      <material name="amr_charcoal"/>
-    </visual>
-    <!-- ── Central identification mast (tapered frustum) ── -->
-    <visual name="mast">
-      <origin xyz="0 0 0" rpy="0 0 0"/>
-      <geometry>
-        <mesh filename="package://warehouse_description/meshes/amr_mast.stl"/>
-      </geometry>
-      <material name="amr_orange"/>
-    </visual>
-    <!-- ── 360° sensor ring (torus) ── -->
-    <visual name="sensor_ring">
-      <origin xyz="0 0 0" rpy="0 0 0"/>
-      <geometry>
-        <mesh filename="package://warehouse_description/meshes/amr_sensor_ring.stl"/>
-      </geometry>
-      <material name="amr_sensor"><color rgba="0.30 0.30 0.30 1.0"/></material>
-    </visual>
-    <!-- ── Safety beacon cylinder ── -->
-    <visual name="beacon_body">
-      <origin xyz="0 0 0" rpy="0 0 0"/>
-      <geometry>
-        <mesh filename="package://warehouse_description/meshes/amr_beacon.stl"/>
-      </geometry>
-      <material name="amr_blue"><color rgba="0.10 0.45 1.00 1.0"/></material>
-    </visual>
-    <!-- ── Safety beacon dome ── -->
-    <visual name="beacon_dome">
-      <origin xyz="0 0 0" rpy="0 0 0"/>
-      <geometry>
-        <mesh filename="package://warehouse_description/meshes/amr_dome.stl"/>
-      </geometry>
-      <material name="amr_blue"/>
-    </visual>
-    <!-- ── Physical collision — full body box ── -->
+    <visual>
+      <origin xyz="0 0 ${body_z}" rpy="0 0 0"/>
+      <geometry><box size="0.900 0.650 0.400"/></geometry>
+    </visual>
     <collision>
       <origin xyz="0 0 ${body_z}" rpy="0 0 0"/>
-      <geometry><box size="0.960 0.660 ${body_h}"/></geometry>
+      <geometry><box size="0.960 0.660 0.400"/></geometry>
     </collision>
     <inertial>
       <origin xyz="0 0 ${body_z}" rpy="0 0 0"/>
       <mass value="${base_mass}"/>
-      <!-- Solid box m=60, l=0.9, w=0.65, h=0.4 -->
       <inertia ixx="2.913" iyy="4.850" izz="6.163"
                ixy="0" ixz="0" iyz="0"/>
     </inertial>
   </link>
-  <!-- ── Left Drive Wheel ── -->
+  <gazebo reference="${robot_ns}/base_link">
+    <material>
+      <ambient>0.90 0.50 0.00 1</ambient>
+      <diffuse>1.00 0.55 0.00 1</diffuse>
+      <specular>0.35 0.22 0.05 1</specular>
+    </material>
+  </gazebo>
+  <!-- ═══════════════════════════════════════════════════════════════════
+       2. TOP LID — charcoal overhanging plate
+       ═══════════════════════════════════════════════════════════════════ -->
+  <xacro:visual_link name="lid_link"/>
+  <xacro:fixed_joint name="lid_jnt" parent="base_link" child="lid_link"
+                     ox="0" oy="0" oz="0.258"/>
+  <link name="${robot_ns}/lid_link">
+    <visual>
+      <origin xyz="0 0 0" rpy="0 0 0"/>
+      <geometry><box size="0.920 0.670 0.026"/></geometry>
+    </visual>
+  </link>
+  <gazebo reference="${robot_ns}/lid_link">
+    <material>
+      <ambient>0.14 0.14 0.14 1</ambient>
+      <diffuse>0.18 0.18 0.18 1</diffuse>
+      <specular>0.12 0.12 0.12 1</specular>
+    </material>
+  </gazebo>
+  <!-- ═══════════════════════════════════════════════════════════════════
+       3. FRONT BUMPER — charcoal safety bar + yellow warning stripe
+       ═══════════════════════════════════════════════════════════════════ -->
+  <xacro:visual_link name="bumper_front_link"/>
+  <xacro:fixed_joint name="bumper_front_jnt" parent="base_link" child="bumper_front_link"
+                     ox="0.481" oy="0" oz="-0.025"/>
+  <link name="${robot_ns}/bumper_front_link">
+    <visual>
+      <origin xyz="0 0 0" rpy="0 0 0"/>
+      <geometry><box size="0.062 0.720 0.260"/></geometry>
+    </visual>
+    <!-- Warning stripe -->
+    <visual>
+      <origin xyz="0.002 0 0.090" rpy="0 0 0"/>
+      <geometry><box size="0.064 0.722 0.042"/></geometry>
+    </visual>
+  </link>
+  <gazebo reference="${robot_ns}/bumper_front_link">
+    <material>
+      <ambient>0.14 0.14 0.14 1</ambient>
+      <diffuse>0.18 0.18 0.18 1</diffuse>
+      <specular>0.12 0.12 0.12 1</specular>
+    </material>
+  </gazebo>
+  <!-- ═══════════════════════════════════════════════════════════════════
+       4. REAR BUMPER
+       ═══════════════════════════════════════════════════════════════════ -->
+  <xacro:visual_link name="bumper_rear_link"/>
+  <xacro:fixed_joint name="bumper_rear_jnt" parent="base_link" child="bumper_rear_link"
+                     ox="-0.481" oy="0" oz="-0.025"/>
+  <link name="${robot_ns}/bumper_rear_link">
+    <visual>
+      <origin xyz="0 0 0" rpy="0 0 0"/>
+      <geometry><box size="0.062 0.720 0.260"/></geometry>
+    </visual>
+    <visual>
+      <origin xyz="-0.002 0 0.090" rpy="0 0 0"/>
+      <geometry><box size="0.064 0.722 0.042"/></geometry>
+    </visual>
+  </link>
+  <gazebo reference="${robot_ns}/bumper_rear_link">
+    <material>
+      <ambient>0.14 0.14 0.14 1</ambient>
+      <diffuse>0.18 0.18 0.18 1</diffuse>
+      <specular>0.12 0.12 0.12 1</specular>
+    </material>
+  </gazebo>
+  <!-- ═══════════════════════════════════════════════════════════════════
+       5. SIDE ACCENT STRIPES — thin dark panels each side
+       ═══════════════════════════════════════════════════════════════════ -->
+  <xacro:visual_link name="accent_left_link"/>
+  <xacro:fixed_joint name="accent_left_jnt" parent="base_link" child="accent_left_link"
+                     ox="0" oy="0.336" oz="0.045"/>
+  <link name="${robot_ns}/accent_left_link">
+    <visual>
+      <origin xyz="0 0 0" rpy="0 0 0"/>
+      <geometry><box size="0.900 0.022 0.400"/></geometry>
+    </visual>
+  </link>
+  <gazebo reference="${robot_ns}/accent_left_link">
+    <material>
+      <ambient>0.14 0.14 0.14 1</ambient>
+      <diffuse>0.18 0.18 0.18 1</diffuse>
+      <specular>0.12 0.12 0.12 1</specular>
+    </material>
+  </gazebo>
+  <xacro:visual_link name="accent_right_link"/>
+  <xacro:fixed_joint name="accent_right_jnt" parent="base_link" child="accent_right_link"
+                     ox="0" oy="-0.336" oz="0.045"/>
+  <link name="${robot_ns}/accent_right_link">
+    <visual>
+      <origin xyz="0 0 0" rpy="0 0 0"/>
+      <geometry><box size="0.900 0.022 0.400"/></geometry>
+    </visual>
+  </link>
+  <gazebo reference="${robot_ns}/accent_right_link">
+    <material>
+      <ambient>0.14 0.14 0.14 1</ambient>
+      <diffuse>0.18 0.18 0.18 1</diffuse>
+      <specular>0.12 0.12 0.12 1</specular>
+    </material>
+  </gazebo>
+  <!-- ═══════════════════════════════════════════════════════════════════
+       6. IDENTIFICATION MAST — orange tapered pole
+       ═══════════════════════════════════════════════════════════════════ -->
+  <xacro:visual_link name="mast_link"/>
+  <xacro:fixed_joint name="mast_jnt" parent="base_link" child="mast_link"
+                     ox="0" oy="0" oz="0.721"/>
+  <link name="${robot_ns}/mast_link">
+    <!-- Lower mast half (thicker) -->
+    <visual>
+      <origin xyz="0 0 -0.225" rpy="0 0 0"/>
+      <geometry><cylinder length="0.450" radius="0.062"/></geometry>
+    </visual>
+    <!-- Upper mast half (thinner — tapered look) -->
+    <visual>
+      <origin xyz="0 0  0.225" rpy="0 0 0"/>
+      <geometry><cylinder length="0.450" radius="0.048"/></geometry>
+    </visual>
+  </link>
+  <gazebo reference="${robot_ns}/mast_link">
+    <material>
+      <ambient>0.90 0.50 0.00 1</ambient>
+      <diffuse>1.00 0.55 0.00 1</diffuse>
+      <specular>0.35 0.22 0.05 1</specular>
+    </material>
+  </gazebo>
+  <!-- ═══════════════════════════════════════════════════════════════════
+       7. 360° SENSOR RING — dark grey housing at mid-mast
+       ═══════════════════════════════════════════════════════════════════ -->
+  <xacro:visual_link name="sensor_ring_link"/>
+  <xacro:fixed_joint name="sensor_ring_jnt" parent="base_link" child="sensor_ring_link"
+                     ox="0" oy="0" oz="0.721"/>
+  <link name="${robot_ns}/sensor_ring_link">
+    <!-- Outer housing disc -->
+    <visual>
+      <origin xyz="0 0 0" rpy="0 0 0"/>
+      <geometry><cylinder length="0.115" radius="0.145"/></geometry>
+    </visual>
+    <!-- Blue sensor window band -->
+    <visual>
+      <origin xyz="0 0 0" rpy="0 0 0"/>
+      <geometry><cylinder length="0.040" radius="0.152"/></geometry>
+    </visual>
+  </link>
+  <gazebo reference="${robot_ns}/sensor_ring_link">
+    <material>
+      <ambient>0.28 0.28 0.28 1</ambient>
+      <diffuse>0.32 0.32 0.32 1</diffuse>
+      <specular>0.18 0.18 0.18 1</specular>
+    </material>
+  </gazebo>
+  <!-- ═══════════════════════════════════════════════════════════════════
+       8. SAFETY BEACON — bright blue cylinder + sphere
+       ═══════════════════════════════════════════════════════════════════ -->
+  <xacro:visual_link name="beacon_link"/>
+  <xacro:fixed_joint name="beacon_jnt" parent="base_link" child="beacon_link"
+                     ox="0" oy="0" oz="1.281"/>
+  <link name="${robot_ns}/beacon_link">
+    <visual>
+      <origin xyz="0 0 0" rpy="0 0 0"/>
+      <geometry><cylinder length="0.200" radius="0.068"/></geometry>
+    </visual>
+  </link>
+  <gazebo reference="${robot_ns}/beacon_link">
+    <material>
+      <ambient>0.05 0.25 1.00 1</ambient>
+      <diffuse>0.10 0.45 1.00 1</diffuse>
+      <specular>0.40 0.60 1.00 1</specular>
+      <emissive>0.01 0.04 0.15 1</emissive>
+    </material>
+  </gazebo>
+  <xacro:visual_link name="dome_link"/>
+  <xacro:fixed_joint name="dome_jnt" parent="base_link" child="dome_link"
+                     ox="0" oy="0" oz="1.471"/>
+  <link name="${robot_ns}/dome_link">
+    <visual>
+      <origin xyz="0 0 0" rpy="0 0 0"/>
+      <geometry><sphere radius="0.090"/></geometry>
+    </visual>
+  </link>
+  <gazebo reference="${robot_ns}/dome_link">
+    <material>
+      <ambient>0.05 0.25 1.00 1</ambient>
+      <diffuse>0.10 0.45 1.00 1</diffuse>
+      <specular>0.40 0.60 1.00 1</specular>
+      <emissive>0.01 0.04 0.15 1</emissive>
+    </material>
+  </gazebo>
+  <!-- ═══════════════════════════════════════════════════════════════════
+       9 & 10. DRIVE WHEELS  (left + right)
+       ═══════════════════════════════════════════════════════════════════ -->
   <joint name="${robot_ns}/wheel_left_joint" type="continuous">
     <parent link="${robot_ns}/base_link"/>
@@ -122,16 +283,17 @@
   </joint>
   <link name="${robot_ns}/wheel_left_link">
-    <visual name="wheel">
-      <origin xyz="0 0 0" rpy="0 0 0"/>
-      <geometry>
-        <mesh filename="package://warehouse_description/meshes/amr_wheel.stl"/>
-      </geometry>
-      <material name="amr_tyre"><color rgba="0.08 0.08 0.08 1.0"/></material>
+    <!-- Tyre -->
+    <visual>
+      <origin xyz="0 0 0" rpy="0 0 0"/>
+      <geometry><cylinder length="${wheel_width}" radius="${wheel_radius}"/></geometry>
+    </visual>
+    <!-- Hub cap -->
+    <visual>
+      <origin xyz="0 0 0.042" rpy="0 0 0"/>
+      <geometry><cylinder length="0.018" radius="0.088"/></geometry>
     </visual>
     <collision>
       <origin xyz="0 0 0" rpy="0 0 0"/>
-      <geometry>
-        <cylinder length="${wheel_width}" radius="${wheel_radius}"/>
-      </geometry>
+      <geometry><cylinder length="${wheel_width}" radius="${wheel_radius}"/></geometry>
     </collision>
     <inertial>
@@ -141,5 +303,7 @@
     </inertial>
   </link>
-  <!-- ── Right Drive Wheel ── -->
+  <gazebo reference="${robot_ns}/wheel_left_link">
+    <material>Gazebo/FlatBlack</material>
+  </gazebo>
   <joint name="${robot_ns}/wheel_right_joint" type="continuous">
     <parent link="${robot_ns}/base_link"/>
@@ -149,16 +313,15 @@
   </joint>
   <link name="${robot_ns}/wheel_right_link">
-    <visual name="wheel">
-      <origin xyz="0 0 0" rpy="0 0 0"/>
-      <geometry>
-        <mesh filename="package://warehouse_description/meshes/amr_wheel.stl"/>
-      </geometry>
-      <material name="amr_tyre"/>
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