Commit message: fix(urdf): remove duplicate link definitions that prevented robot spawning
The xacro:visual_link macro was creating a <link> with only <inertial>,
then a second <link> with the same namespaced name containing only <visual>.
URDF parsers reject duplicate link names, causing robot_state_publisher
to fail and all four robots to be invisible in Gazebo.

Fix: delete the visual_link macro entirely and write each decoration link
as a single complete <link> with both <visual> and <inertial> blocks.
All 17 links are now unique; xacro expansion is verified clean.

Co-Authored-By: Claude Sonnet 4.6 <noreply@anthropic.com>
Claude-Session: https://claude.ai/code/session_016EwupYKQVrfCeF8yG8S6Li

File: src/warehouse_description/urdf/warehouse_robot.urdf.xacro (robot description, xacro)
@@ -22,27 +22,8 @@
   <xacro:property name="caster_front_x"  value=" 0.395"/>
   <xacro:property name="caster_rear_x"   value="-0.395"/>
-  <!-- Pre-computed geometry constants (base_link frame) -->
-  <!-- body_bottom = -0.175 + 0.020(clearance) = -0.155                  -->
-  <!-- body_z      = -0.155 + 0.200             =  0.045  (body centre)   -->
-  <!-- body_top    =  0.045 + 0.200             =  0.245                  -->
-  <!-- lid_cz      =  0.245 + 0.013             =  0.258                  -->
-  <!-- bumper_cz   = -0.155 + 0.130             = -0.025                  -->
-  <!-- mast_cz     =  0.271 + 0.450             =  0.721  (mast centre)   -->
-  <!-- beacon_cz   =  1.171 + 0.110             =  1.281                  -->
-  <!-- dome_cz     =  1.281 + 0.100 + 0.090     =  1.471                  -->
+  <!-- body_z = body centre in base_link frame -->
   <xacro:property name="body_z"   value=" 0.045"/>
   <xacro:property name="body_h"   value=" 0.400"/>
-  <!-- ════════════════════════════════════════
-       Helper macro: inertia-free visual link
-       (used for all decoration-only links)
-       ════════════════════════════════════════ -->
-  <xacro:macro name="visual_link" params="name">
-    <link name="${robot_ns}/${name}">
-      <inertial>
-        <mass value="0.001"/>
-        <inertia ixx="1e-9" iyy="1e-9" izz="1e-9" ixy="0" ixz="0" iyz="0"/>
-      </inertial>
-    </link>
-  </xacro:macro>
+  <!-- Helper macro: fixed joint only (no visual_link macro — links defined inline) -->
   <xacro:macro name="fixed_joint" params="name parent child ox oy oz">
     <joint name="${robot_ns}/${name}" type="fixed">
@@ -88,5 +69,4 @@
        2. TOP LID — charcoal overhanging plate
        ═══════════════════════════════════════════════════════════════════ -->
-  <xacro:visual_link name="lid_link"/>
   <xacro:fixed_joint name="lid_jnt" parent="base_link" child="lid_link"
                      ox="0" oy="0" oz="0.258"/>
@@ -96,4 +76,8 @@
       <geometry><box size="0.920 0.670 0.026"/></geometry>
     </visual>
+    <inertial>
+      <mass value="0.001"/>
+      <inertia ixx="1e-9" iyy="1e-9" izz="1e-9" ixy="0" ixz="0" iyz="0"/>
+    </inertial>
   </link>
   <gazebo reference="${robot_ns}/lid_link">
@@ -107,5 +91,4 @@
        3. FRONT BUMPER — charcoal safety bar + yellow warning stripe
        ═══════════════════════════════════════════════════════════════════ -->
-  <xacro:visual_link name="bumper_front_link"/>
   <xacro:fixed_joint name="bumper_front_jnt" parent="base_link" child="bumper_front_link"
                      ox="0.481" oy="0" oz="-0.025"/>
@@ -115,9 +98,12 @@
       <geometry><box size="0.062 0.720 0.260"/></geometry>
     </visual>
-    <!-- Warning stripe -->
     <visual>
       <origin xyz="0.002 0 0.090" rpy="0 0 0"/>
       <geometry><box size="0.064 0.722 0.042"/></geometry>
     </visual>
+    <inertial>
+      <mass value="0.001"/>
+      <inertia ixx="1e-9" iyy="1e-9" izz="1e-9" ixy="0" ixz="0" iyz="0"/>
+    </inertial>
   </link>
   <gazebo reference="${robot_ns}/bumper_front_link">
@@ -131,5 +117,4 @@
        4. REAR BUMPER
        ═══════════════════════════════════════════════════════════════════ -->
-  <xacro:visual_link name="bumper_rear_link"/>
   <xacro:fixed_joint name="bumper_rear_jnt" parent="base_link" child="bumper_rear_link"
                      ox="-0.481" oy="0" oz="-0.025"/>
@@ -143,4 +128,8 @@
       <geometry><box size="0.064 0.722 0.042"/></geometry>
     </visual>
+    <inertial>
+      <mass value="0.001"/>
+      <inertia ixx="1e-9" iyy="1e-9" izz="1e-9" ixy="0" ixz="0" iyz="0"/>
+    </inertial>
   </link>
   <gazebo reference="${robot_ns}/bumper_rear_link">
@@ -154,5 +143,4 @@
        5. SIDE ACCENT STRIPES — thin dark panels each side
        ═══════════════════════════════════════════════════════════════════ -->
-  <xacro:visual_link name="accent_left_link"/>
   <xacro:fixed_joint name="accent_left_jnt" parent="base_link" child="accent_left_link"
                      ox="0" oy="0.336" oz="0.045"/>
@@ -162,4 +150,8 @@
       <geometry><box size="0.900 0.022 0.400"/></geometry>
     </visual>
+    <inertial>
+      <mass value="0.001"/>
+      <inertia ixx="1e-9" iyy="1e-9" izz="1e-9" ixy="0" ixz="0" iyz="0"/>
+    </inertial>
   </link>
   <gazebo reference="${robot_ns}/accent_left_link">
@@ -170,5 +162,4 @@
     </material>
   </gazebo>
-  <xacro:visual_link name="accent_right_link"/>
   <xacro:fixed_joint name="accent_right_jnt" parent="base_link" child="accent_right_link"
                      ox="0" oy="-0.336" oz="0.045"/>
@@ -178,4 +169,8 @@
       <geometry><box size="0.900 0.022 0.400"/></geometry>
     </visual>
+    <inertial>
+      <mass value="0.001"/>
+      <inertia ixx="1e-9" iyy="1e-9" izz="1e-9" ixy="0" ixz="0" iyz="0"/>
+    </inertial>
   </link>
   <gazebo reference="${robot_ns}/accent_right_link">
@@ -189,18 +184,19 @@
        6. IDENTIFICATION MAST — orange tapered pole
        ═══════════════════════════════════════════════════════════════════ -->
-  <xacro:visual_link name="mast_link"/>
   <xacro:fixed_joint name="mast_jnt" parent="base_link" child="mast_link"
                      ox="0" oy="0" oz="0.721"/>
   <link name="${robot_ns}/mast_link">
-    <!-- Lower mast half (thicker) -->
     <visual>
       <origin xyz="0 0 -0.225" rpy="0 0 0"/>
       <geometry><cylinder length="0.450" radius="0.062"/></geometry>
     </visual>
-    <!-- Upper mast half (thinner — tapered look) -->
     <visual>
       <origin xyz="0 0  0.225" rpy="0 0 0"/>
       <geometry><cylinder length="0.450" radius="0.048"/></geometry>
     </visual>
+    <inertial>
+      <mass value="0.001"/>
+      <inertia ixx="1e-9" iyy="1e-9" izz="1e-9" ixy="0" ixz="0" iyz="0"/>
+    </inertial>
   </link>
   <gazebo reference="${robot_ns}/mast_link">
@@ -214,18 +210,19 @@
        7. 360° SENSOR RING — dark grey housing at mid-mast
        ═══════════════════════════════════════════════════════════════════ -->
-  <xacro:visual_link name="sensor_ring_link"/>
   <xacro:fixed_joint name="sensor_ring_jnt" parent="base_link" child="sensor_ring_link"
                      ox="0" oy="0" oz="0.721"/>
   <link name="${robot_ns}/sensor_ring_link">
-    <!-- Outer housing disc -->
     <visual>
       <origin xyz="0 0 0" rpy="0 0 0"/>
       <geometry><cylinder length="0.115" radius="0.145"/></geometry>
     </visual>
-    <!-- Blue sensor window band -->
     <visual>
       <origin xyz="0 0 0" rpy="0 0 0"/>
       <geometry><cylinder length="0.040" radius="0.152"/></geometry>
     </visual>
+    <inertial>
+      <mass value="0.001"/>
+      <inertia ixx="1e-9" iyy="1e-9" izz="1e-9" ixy="0" ixz="0" iyz="0"/>
+    </inertial>
   </link>
   <gazebo reference="${robot_ns}/sensor_ring_link">
@@ -237,7 +234,6 @@
   </gazebo>
   <!-- ═══════════════════════════════════════════════════════════════════
-       8. SAFETY BEACON — bright blue cylinder + sphere
-       ═══════════════════════════════════════════════════════════════════ -->
-  <xacro:visual_link name="beacon_link"/>
+       8. SAFETY BEACON — bright blue cylinder
+       ═══════════════════════════════════════════════════════════════════ -->
   <xacro:fixed_joint name="beacon_jnt" parent="base_link" child="beacon_link"
                      ox="0" oy="0" oz="1.281"/>
@@ -247,4 +243,8 @@
       <geometry><cylinder length="0.200" radius="0.068"/></geometry>
     </visual>
+    <inertial>
+      <mass value="0.001"/>
+      <inertia ixx="1e-9" iyy="1e-9" izz="1e-9" ixy="0" ixz="0" iyz="0"/>
+    </inertial>
   </link>
   <gazebo reference="${robot_ns}/beacon_link">
@@ -256,5 +256,7 @@
     </material>
   </gazebo>
-  <xacro:visual_link name="dome_link"/>
+  <!-- ═══════════════════════════════════════════════════════════════════
+       9. BEACON DOME — blue sphere on top
+       ═══════════════════════════════════════════════════════════════════ -->
   <xacro:fixed_joint name="dome_jnt" parent="base_link" child="dome_link"
                      ox="0" oy="0" oz="1.471"/>
@@ -264,4 +266,8 @@
       <geometry><sphere radius="0.090"/></geometry>
     </visual>
+    <inertial>
+      <mass value="0.001"/>
+      <inertia ixx="1e-9" iyy="1e-9" izz="1e-9" ixy="0" ixz="0" iyz="0"/>
+    </inertial>
   </link>
   <gazebo reference="${robot_ns}/dome_link">
@@ -274,5 +280,5 @@
   </gazebo>
   <!-- ═══════════════════════════════════════════════════════════════════
-       9 & 10. DRIVE WHEELS  (left + right)
+       10 & 11. DRIVE WHEELS  (left + right)
        ═══════════════════════════════════════════════════════════════════ -->
   <joint name="${robot_ns}/wheel_left_joint" type="continuous">
@@ -283,10 +289,8 @@
   </joint>
   <link name="${robot_ns}/wheel_left_link">
-    <!-- Tyre -->
     <visual>
       <origin xyz="0 0 0" rpy="0 0 0"/>
       <geometry><cylinder length="${wheel_width}" radius="${wheel_radius}"/></geometry>
     </visual>
-    <!-- Hub cap -->
     <visual>
       <origin xyz="0 0 0.042" rpy="0 0 0"/>
@@ -335,5 +339,5 @@
   </gazebo>
   <!-- ═══════════════════════════════════════════════════════════════════
-       11 & 12. CASTER BALLS (front + rear)
+       12 & 13. CASTER BALLS (front + rear)
        ═══════════════════════════════════════════════════════════════════ -->
   <joint name="${robot_ns}/caster_front_joint" type="fixed">
@@ -370,5 +374,5 @@
   </gazebo>
   <!-- ═══════════════════════════════════════════════════════════════════
-       13. LiDAR  (at sensor-ring height — 0.896 m above ground)
+       14. LiDAR  (at sensor-ring height — 0.896 m above ground)
        ═══════════════════════════════════════════════════════════════════ -->
   <xacro:if value="$(arg laser_enable)">
@@ -421,5 +425,5 @@
   </xacro:if>
   <!-- ═══════════════════════════════════════════════════════════════════
-       14. IMU
+       15. IMU
        ═══════════════════════════════════════════════════════════════════ -->
   <xacro:if value="$(arg imu_enable)">
