Commit message: feat: replace robot with TurtleBot3 Burger model
Switch robot to TurtleBot3 Burger-style model:
- Two circular plates (dark grey, r=0.105m) with 4 standoff poles
- Small black drive wheels (r=0.033m, separation=0.160m)
- Two low-friction caster balls
- LiDAR housing cylinder on top plate
- Diff drive plugin tuned for TB3 (torque=5 Nm, accel=50 rad/s²)
- Spawn height updated to 0.033m (wheel radius)
- Fleet manager MAX_LIN tuned to 1.5 m/s for TurtleBot3

Co-Authored-By: Claude Sonnet 4.6 <noreply@anthropic.com>
Claude-Session: https://claude.ai/code/session_016EwupYKQVrfCeF8yG8S6Li

File: src/warehouse_description/urdf/warehouse_robot.urdf.xacro (robot description, xacro)
@@ -9,21 +9,27 @@
   <xacro:property name="robot_ns" value="$(arg robot_name)"/>
   <!-- ═══════════════════════════════════════════════════════════════════
-       PHYSICS  — spawn height z = 0.175 m  (= wheel_radius + |offset|)
-       Ground plane is at base_link z = −0.175 m
-       ═══════════════════════════════════════════════════════════════════ -->
-  <xacro:property name="base_mass"       value="60.0"/>
-  <xacro:property name="wheel_radius"    value="0.170"/>
-  <xacro:property name="wheel_width"     value="0.080"/>
-  <xacro:property name="wheel_sep_half"  value="0.290"/>   <!-- 0.580 m axle / 2 -->
-  <xacro:property name="wheel_offset_z"  value="-0.005"/>
-  <xacro:property name="caster_radius"   value="0.050"/>
-  <!-- caster bottom must touch ground: caster_z = caster_radius − spawn_z = 0.050−0.175 -->
-  <xacro:property name="caster_z"        value="-0.125"/>
-  <xacro:property name="caster_front_x"  value=" 0.395"/>
-  <xacro:property name="caster_rear_x"   value="-0.395"/>
-  <!-- body_z = body centre in base_link frame -->
-  <xacro:property name="body_z"   value=" 0.045"/>
-  <xacro:property name="body_h"   value=" 0.400"/>
-  <!-- Helper macro: fixed joint only (no visual_link macro — links defined inline) -->
+       TurtleBot3 Burger dimensions
+       spawn height z = 0.033 m  (= wheel_radius)
+       base_link frame origin  = wheel axle height
+       ground plane at         = z − 0.033 m in base_link frame
+       ═══════════════════════════════════════════════════════════════════ -->
+  <xacro:property name="base_mass"      value="1.0"/>
+  <xacro:property name="wheel_radius"   value="0.033"/>
+  <xacro:property name="wheel_width"    value="0.018"/>
+  <xacro:property name="wheel_sep_half" value="0.080"/>   <!-- 0.160 m / 2 -->
+  <xacro:property name="caster_radius"  value="0.010"/>
+  <!-- Positions in base_link frame (ground = −0.033) -->
+  <!-- bottom plate centre: 0.010 m above ground → −0.033+0.010+0.0035 = −0.0195 -->
+  <xacro:property name="bottom_plate_z" value="-0.020"/>
+  <!-- top plate centre: 0.190 m above ground → −0.033+0.190+0.0035 = 0.1605 -->
+  <xacro:property name="top_plate_z"    value="0.161"/>
+  <!-- standoff centre (midpoint between plates) -->
+  <xacro:property name="standoff_z"     value="0.071"/>
+  <xacro:property name="standoff_len"   value="0.174"/>
+  <!-- lidar base just above top plate -->
+  <xacro:property name="lidar_z"        value="0.185"/>
+  <!-- casters: bottom touches ground → centre at −0.033+caster_radius -->
+  <xacro:property name="caster_z"       value="-0.023"/>
+  <!-- Helper: fixed joint -->
   <xacro:macro name="fixed_joint" params="name parent child ox oy oz">
     <joint name="${robot_ns}/${name}" type="fixed">
@@ -41,19 +47,21 @@
   </joint>
   <!-- ═══════════════════════════════════════════════════════════════════
-       1. BASE LINK — orange body box + collision + inertia
+       1. BASE LINK — bottom circular plate + physics
        ═══════════════════════════════════════════════════════════════════ -->
   <link name="${robot_ns}/base_link">
     <visual>
-      <origin xyz="0 0 ${body_z}" rpy="0 0 0"/>
-      <geometry><box size="0.900 0.650 0.400"/></geometry>
+      <origin xyz="0 0 ${bottom_plate_z}" rpy="0 0 0"/>
+      <geometry><cylinder length="0.007" radius="0.105"/></geometry>
     </visual>
     <collision>
-      <origin xyz="0 0 ${body_z}" rpy="0 0 0"/>
-      <geometry><box size="0.960 0.660 0.400"/></geometry>
+      <!-- Flat cylinder collision to keep robot on ground -->
+      <origin xyz="0 0 ${bottom_plate_z}" rpy="0 0 0"/>
+      <geometry><cylinder length="0.100" radius="0.105"/></geometry>
     </collision>
     <inertial>
-      <origin xyz="0 0 ${body_z}" rpy="0 0 0"/>
+      <origin xyz="0 0 ${bottom_plate_z}" rpy="0 0 0"/>
       <mass value="${base_mass}"/>
-      <inertia ixx="2.913" iyy="4.850" izz="6.163"
+      <!-- Thin cylinder: Ixx=Iyy=m(3r²+h²)/12, Izz=mr²/2 -->
+      <inertia ixx="0.00277" iyy="0.00277" izz="0.00551"
                ixy="0" ixz="0" iyz="0"/>
     </inertial>
@@ -61,229 +69,139 @@
   <gazebo reference="${robot_ns}/base_link">
     <material>
-      <ambient>0.90 0.50 0.00 1</ambient>
-      <diffuse>1.00 0.55 0.00 1</diffuse>
-      <specular>0.35 0.22 0.05 1</specular>
-    </material>
-  </gazebo>
-  <!-- ═══════════════════════════════════════════════════════════════════
-       2. TOP LID — charcoal overhanging plate
-       ═══════════════════════════════════════════════════════════════════ -->
-  <xacro:fixed_joint name="lid_jnt" parent="base_link" child="lid_link"
-                     ox="0" oy="0" oz="0.258"/>
-  <link name="${robot_ns}/lid_link">
-    <visual>
-      <origin xyz="0 0 0" rpy="0 0 0"/>
-      <geometry><box size="0.920 0.670 0.026"/></geometry>
-    </visual>
-    <inertial>
-      <mass value="0.001"/>
-      <inertia ixx="1e-9" iyy="1e-9" izz="1e-9" ixy="0" ixz="0" iyz="0"/>
-    </inertial>
-  </link>
-  <gazebo reference="${robot_ns}/lid_link">
-    <material>
-      <ambient>0.14 0.14 0.14 1</ambient>
-      <diffuse>0.18 0.18 0.18 1</diffuse>
-      <specular>0.12 0.12 0.12 1</specular>
-    </material>
-  </gazebo>
-  <!-- ═══════════════════════════════════════════════════════════════════
-       3. FRONT BUMPER — charcoal safety bar + yellow warning stripe
-       ═══════════════════════════════════════════════════════════════════ -->
-  <xacro:fixed_joint name="bumper_front_jnt" parent="base_link" child="bumper_front_link"
-                     ox="0.481" oy="0" oz="-0.025"/>
-  <link name="${robot_ns}/bumper_front_link">
-    <visual>
-      <origin xyz="0 0 0" rpy="0 0 0"/>
-      <geometry><box size="0.062 0.720 0.260"/></geometry>
-    </visual>
-    <visual>
-      <origin xyz="0.002 0 0.090" rpy="0 0 0"/>
-      <geometry><box size="0.064 0.722 0.042"/></geometry>
-    </visual>
-    <inertial>
-      <mass value="0.001"/>
-      <inertia ixx="1e-9" iyy="1e-9" izz="1e-9" ixy="0" ixz="0" iyz="0"/>
-    </inertial>
-  </link>
-  <gazebo reference="${robot_ns}/bumper_front_link">
-    <material>
-      <ambient>0.14 0.14 0.14 1</ambient>
-      <diffuse>0.18 0.18 0.18 1</diffuse>
-      <specular>0.12 0.12 0.12 1</specular>
-    </material>
-  </gazebo>
-  <!-- ═══════════════════════════════════════════════════════════════════
-       4. REAR BUMPER
-       ═══════════════════════════════════════════════════════════════════ -->
-  <xacro:fixed_joint name="bumper_rear_jnt" parent="base_link" child="bumper_rear_link"
-                     ox="-0.481" oy="0" oz="-0.025"/>
-  <link name="${robot_ns}/bumper_rear_link">
-    <visual>
-      <origin xyz="0 0 0" rpy="0 0 0"/>
-      <geometry><box size="0.062 0.720 0.260"/></geometry>
-    </visual>
-    <visual>
-      <origin xyz="-0.002 0 0.090" rpy="0 0 0"/>
-      <geometry><box size="0.064 0.722 0.042"/></geometry>
-    </visual>
-    <inertial>
-      <mass value="0.001"/>
-      <inertia ixx="1e-9" iyy="1e-9" izz="1e-9" ixy="0" ixz="0" iyz="0"/>
-    </inertial>
-  </link>
-  <gazebo reference="${robot_ns}/bumper_rear_link">
-    <material>
-      <ambient>0.14 0.14 0.14 1</ambient>
-      <diffuse>0.18 0.18 0.18 1</diffuse>
-      <specular>0.12 0.12 0.12 1</specular>
-    </material>
-  </gazebo>
-  <!-- ═══════════════════════════════════════════════════════════════════
-       5. SIDE ACCENT STRIPES — thin dark panels each side
-       ═══════════════════════════════════════════════════════════════════ -->
-  <xacro:fixed_joint name="accent_left_jnt" parent="base_link" child="accent_left_link"
-                     ox="0" oy="0.336" oz="0.045"/>
-  <link name="${robot_ns}/accent_left_link">
-    <visual>
-      <origin xyz="0 0 0" rpy="0 0 0"/>
-      <geometry><box size="0.900 0.022 0.400"/></geometry>
-    </visual>
-    <inertial>
-      <mass value="0.001"/>
-      <inertia ixx="1e-9" iyy="1e-9" izz="1e-9" ixy="0" ixz="0" iyz="0"/>
-    </inertial>
-  </link>
-  <gazebo reference="${robot_ns}/accent_left_link">
-    <material>
-      <ambient>0.14 0.14 0.14 1</ambient>
-      <diffuse>0.18 0.18 0.18 1</diffuse>
-      <specular>0.12 0.12 0.12 1</specular>
-    </material>
-  </gazebo>
-  <xacro:fixed_joint name="accent_right_jnt" parent="base_link" child="accent_right_link"
-                     ox="0" oy="-0.336" oz="0.045"/>
-  <link name="${robot_ns}/accent_right_link">
-    <visual>
-      <origin xyz="0 0 0" rpy="0 0 0"/>
-      <geometry><box size="0.900 0.022 0.400"/></geometry>
-    </visual>
-    <inertial>
-      <mass value="0.001"/>
-      <inertia ixx="1e-9" iyy="1e-9" izz="1e-9" ixy="0" ixz="0" iyz="0"/>
-    </inertial>
-  </link>
-  <gazebo reference="${robot_ns}/accent_right_link">
-    <material>
-      <ambient>0.14 0.14 0.14 1</ambient>
-      <diffuse>0.18 0.18 0.18 1</diffuse>
-      <specular>0.12 0.12 0.12 1</specular>
-    </material>
-  </gazebo>
-  <!-- ═══════════════════════════════════════════════════════════════════
-       6. IDENTIFICATION MAST — orange tapered pole
-       ═══════════════════════════════════════════════════════════════════ -->
-  <xacro:fixed_joint name="mast_jnt" parent="base_link" child="mast_link"
-                     ox="0" oy="0" oz="0.721"/>
-  <link name="${robot_ns}/mast_link">
-    <visual>
-      <origin xyz="0 0 -0.225" rpy="0 0 0"/>
-      <geometry><cylinder length="0.450" radius="0.062"/></geometry>
-    </visual>
-    <visual>
-      <origin xyz="0 0  0.225" rpy="0 0 0"/>
-      <geometry><cylinder length="0.450" radius="0.048"/></geometry>
-    </visual>
-    <inertial>
-      <mass value="0.001"/>
-      <inertia ixx="1e-9" iyy="1e-9" izz="1e-9" ixy="0" ixz="0" iyz="0"/>
-    </inertial>
-  </link>
-  <gazebo reference="${robot_ns}/mast_link">
-    <material>
-      <ambient>0.90 0.50 0.00 1</ambient>
-      <diffuse>1.00 0.55 0.00 1</diffuse>
-      <specular>0.35 0.22 0.05 1</specular>
-    </material>
-  </gazebo>
-  <!-- ═══════════════════════════════════════════════════════════════════
-       7. 360° SENSOR RING — dark grey housing at mid-mast
-       ═══════════════════════════════════════════════════════════════════ -->
-  <xacro:fixed_joint name="sensor_ring_jnt" parent="base_link" child="sensor_ring_link"
-                     ox="0" oy="0" oz="0.721"/>
-  <link name="${robot_ns}/sensor_ring_link">
-    <visual>
-      <origin xyz="0 0 0" rpy="0 0 0"/>
-      <geometry><cylinder length="0.115" radius="0.145"/></geometry>
-    </visual>
-    <visual>
-      <origin xyz="0 0 0" rpy="0 0 0"/>
-      <geometry><cylinder length="0.040" radius="0.152"/></geometry>
-    </visual>
-    <inertial>
-      <mass value="0.001"/>
-      <inertia ixx="1e-9" iyy="1e-9" izz="1e-9" ixy="0" ixz="0" iyz="0"/>
-    </inertial>
-  </link>
-  <gazebo reference="${robot_ns}/sensor_ring_link">
-    <material>
-      <ambient>0.28 0.28 0.28 1</ambient>
-      <diffuse>0.32 0.32 0.32 1</diffuse>
-      <specular>0.18 0.18 0.18 1</specular>
-    </material>
-  </gazebo>
-  <!-- ═══════════════════════════════════════════════════════════════════
-       8. SAFETY BEACON — bright blue cylinder
-       ═══════════════════════════════════════════════════════════════════ -->
-  <xacro:fixed_joint name="beacon_jnt" parent="base_link" child="beacon_link"
-                     ox="0" oy="0" oz="1.281"/>
-  <link name="${robot_ns}/beacon_link">
-    <visual>
-      <origin xyz="0 0 0" rpy="0 0 0"/>
-      <geometry><cylinder length="0.200" radius="0.068"/></geometry>
-    </visual>
-    <inertial>
-      <mass value="0.001"/>
-      <inertia ixx="1e-9" iyy="1e-9" izz="1e-9" ixy="0" ixz="0" iyz="0"/>
-    </inertial>
-  </link>
-  <gazebo reference="${robot_ns}/beacon_link">
-    <material>
-      <ambient>0.05 0.25 1.00 1</ambient>
-      <diffuse>0.10 0.45 1.00 1</diffuse>
-      <specular>0.40 0.60 1.00 1</specular>
-      <emissive>0.01 0.04 0.15 1</emissive>
-    </material>
-  </gazebo>
-  <!-- ═══════════════════════════════════════════════════════════════════
-       9. BEACON DOME — blue sphere on top
-       ═══════════════════════════════════════════════════════════════════ -->
-  <xacro:fixed_joint name="dome_jnt" parent="base_link" child="dome_link"
-                     ox="0" oy="0" oz="1.471"/>
-  <link name="${robot_ns}/dome_link">
-    <visual>
-      <origin xyz="0 0 0" rpy="0 0 0"/>
-      <geometry><sphere radius="0.090"/></geometry>
-    </visual>
-    <inertial>
-      <mass value="0.001"/>
-      <inertia ixx="1e-9" iyy="1e-9" izz="1e-9" ixy="0" ixz="0" iyz="0"/>
-    </inertial>
-  </link>
-  <gazebo reference="${robot_ns}/dome_link">
-    <material>
-      <ambient>0.05 0.25 1.00 1</ambient>
-      <diffuse>0.10 0.45 1.00 1</diffuse>
-      <specular>0.40 0.60 1.00 1</specular>
-      <emissive>0.01 0.04 0.15 1</emissive>
-    </material>
-  </gazebo>
-  <!-- ═══════════════════════════════════════════════════════════════════
-       10 & 11. DRIVE WHEELS  (left + right)
+      <ambient>0.18 0.18 0.18 1</ambient>
+      <diffuse>0.22 0.22 0.22 1</diffuse>
+      <specular>0.10 0.10 0.10 1</specular>
+    </material>
+  </gazebo>
+  <!-- ═══════════════════════════════════════════════════════════════════
+       2. TOP PLATE — second circular plate
+       ═══════════════════════════════════════════════════════════════════ -->
+  <xacro:fixed_joint name="top_plate_jnt" parent="base_link" child="top_plate_link"
+                     ox="0" oy="0" oz="0"/>
+  <link name="${robot_ns}/top_plate_link">
+    <visual>
+      <origin xyz="0 0 ${top_plate_z}" rpy="0 0 0"/>
+      <geometry><cylinder length="0.007" radius="0.105"/></geometry>
+    </visual>
+    <inertial>
+      <mass value="0.001"/>
+      <inertia ixx="1e-9" iyy="1e-9" izz="1e-9" ixy="0" ixz="0" iyz="0"/>
+    </inertial>
+  </link>
+  <gazebo reference="${robot_ns}/top_plate_link">
+    <material>
+      <ambient>0.18 0.18 0.18 1</ambient>
+      <diffuse>0.22 0.22 0.22 1</diffuse>
+      <specular>0.10 0.10 0.10 1</specular>
+    </material>
+  </gazebo>
+  <!-- ═══════════════════════════════════════════════════════════════════
+       3–6. STANDOFF POLES (front-left, front-right, rear-left, rear-right)
+       ═══════════════════════════════════════════════════════════════════ -->
+  <xacro:fixed_joint name="standoff_fl_jnt" parent="base_link" child="standoff_fl_link"
+                     ox="0.055" oy="0.055" oz="${standoff_z}"/>
+  <link name="${robot_ns}/standoff_fl_link">
+    <visual>
+      <origin xyz="0 0 0" rpy="0 0 0"/>
+      <geometry><cylinder length="${standoff_len}" radius="0.011"/></geometry>
+    </visual>
+    <inertial>
+      <mass value="0.001"/>
+      <inertia ixx="1e-9" iyy="1e-9" izz="1e-9" ixy="0" ixz="0" iyz="0"/>
+    </inertial>
+  </link>
+  <gazebo reference="${robot_ns}/standoff_fl_link">
+    <material>
+      <ambient>0.18 0.18 0.18 1</ambient>
+      <diffuse>0.22 0.22 0.22 1</diffuse>
+      <specular>0.10 0.10 0.10 1</specular>
+    </material>
+  </gazebo>
+  <xacro:fixed_joint name="standoff_fr_jnt" parent="base_link" child="standoff_fr_link"
+                     ox="0.055" oy="-0.055" oz="${standoff_z}"/>
+  <link name="${robot_ns}/standoff_fr_link">
+    <visual>
+      <origin xyz="0 0 0" rpy="0 0 0"/>
+      <geometry><cylinder length="${standoff_len}" radius="0.011"/></geometry>
+    </visual>
+    <inertial>
+      <mass value="0.001"/>
+      <inertia ixx="1e-9" iyy="1e-9" izz="1e-9" ixy="0" ixz="0" iyz="0"/>
+    </inertial>
+  </link>
+  <gazebo reference="${robot_ns}/standoff_fr_link">
+    <material>
+      <ambient>0.18 0.18 0.18 1</ambient>
+      <diffuse>0.22 0.22 0.22 1</diffuse>
+      <specular>0.10 0.10 0.10 1</specular>
+    </material>
+  </gazebo>
+  <xacro:fixed_joint name="standoff_rl_jnt" parent="base_link" child="standoff_rl_link"
+                     ox="-0.055" oy="0.055" oz="${standoff_z}"/>
+  <link name="${robot_ns}/standoff_rl_link">
+    <visual>
+      <origin xyz="0 0 0" rpy="0 0 0"/>
+      <geometry><cylinder length="${standoff_len}" radius="0.011"/></geometry>
+    </visual>
+    <inertial>
+      <mass value="0.001"/>
+      <inertia ixx="1e-9" iyy="1e-9" izz="1e-9" ixy="0" ixz="0" iyz="0"/>
+    </inertial>
+  </link>
+  <gazebo reference="${robot_ns}/standoff_rl_link">
+    <material>
+      <ambient>0.18 0.18 0.18 1</ambient>
+      <diffuse>0.22 0.22 0.22 1</diffuse>
+      <specular>0.10 0.10 0.10 1</specular>
+    </material>
+  </gazebo>
+  <xacro:fixed_joint name="standoff_rr_jnt" parent="base_link" child="standoff_rr_link"
+                     ox="-0.055" oy="-0.055" oz="${standoff_z}"/>
+  <link name="${robot_ns}/standoff_rr_link">
+    <visual>
+      <origin xyz="0 0 0" rpy="0 0 0"/>
+      <geometry><cylinder length="${standoff_len}" radius="0.011"/></geometry>
+    </visual>
+    <inertial>
+      <mass value="0.001"/>
+      <inertia ixx="1e-9" iyy="1e-9" izz="1e-9" ixy="0" ixz="0" iyz="0"/>
+    </inertial>
+  </link>
+  <gazebo reference="${robot_ns}/standoff_rr_link">
+    <material>
+      <ambient>0.18 0.18 0.18 1</ambient>
+      <diffuse>0.22 0.22 0.22 1</diffuse>
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
Commit message: fix(urdf): use Gazebo named materials for correct dark-grey colouring
OGRE ambient/diffuse values inside <gazebo reference> were washing out
to near-white in Gazebo Classic renderer. Switch to named materials:
  body plates + standoffs → Gazebo/DarkGrey
  lidar housing           → Gazebo/Black
  wheels                  → Gazebo/FlatBlack  (unchanged)
  casters                 → Gazebo/Grey       (unchanged)

Co-Authored-By: Claude Sonnet 4.6 <noreply@anthropic.com>
Claude-Session: https://claude.ai/code/session_016EwupYKQVrfCeF8yG8S6Li

File: src/warehouse_description/urdf/warehouse_robot.urdf.xacro (robot description, xacro)
@@ -68,9 +68,5 @@
   </link>
   <gazebo reference="${robot_ns}/base_link">
-    <material>
-      <ambient>0.18 0.18 0.18 1</ambient>
-      <diffuse>0.22 0.22 0.22 1</diffuse>
-      <specular>0.10 0.10 0.10 1</specular>
-    </material>
+    <material>Gazebo/DarkGrey</material>
   </gazebo>
   <!-- ═══════════════════════════════════════════════════════════════════
@@ -90,9 +86,5 @@
   </link>
   <gazebo reference="${robot_ns}/top_plate_link">
-    <material>
-      <ambient>0.18 0.18 0.18 1</ambient>
-      <diffuse>0.22 0.22 0.22 1</diffuse>
-      <specular>0.10 0.10 0.10 1</specular>
-    </material>
+    <material>Gazebo/DarkGrey</material>
   </gazebo>
   <!-- ═══════════════════════════════════════════════════════════════════
@@ -112,9 +104,5 @@
   </link>
   <gazebo reference="${robot_ns}/standoff_fl_link">
-    <material>
-      <ambient>0.18 0.18 0.18 1</ambient>
-      <diffuse>0.22 0.22 0.22 1</diffuse>
-      <specular>0.10 0.10 0.10 1</specular>
-    </material>
+    <material>Gazebo/DarkGrey</material>
   </gazebo>
   <xacro:fixed_joint name="standoff_fr_jnt" parent="base_link" child="standoff_fr_link"
@@ -131,9 +119,5 @@
   </link>
   <gazebo reference="${robot_ns}/standoff_fr_link">
-    <material>
-      <ambient>0.18 0.18 0.18 1</ambient>
-      <diffuse>0.22 0.22 0.22 1</diffuse>
-      <specular>0.10 0.10 0.10 1</specular>
-    </material>
+    <material>Gazebo/DarkGrey</material>
   </gazebo>
   <xacro:fixed_joint name="standoff_rl_jnt" parent="base_link" child="standoff_rl_link"
@@ -150,9 +134,5 @@
   </link>
   <gazebo reference="${robot_ns}/standoff_rl_link">
-    <material>
-      <ambient>0.18 0.18 0.18 1</ambient>
-      <diffuse>0.22 0.22 0.22 1</diffuse>
-      <specular>0.10 0.10 0.10 1</specular>
-    </material>
+    <material>Gazebo/DarkGrey</material>
   </gazebo>
   <xacro:fixed_joint name="standoff_rr_jnt" parent="base_link" child="standoff_rr_link"
@@ -169,9 +149,5 @@
   </link>
   <gazebo reference="${robot_ns}/standoff_rr_link">
-    <material>
-      <ambient>0.18 0.18 0.18 1</ambient>
-      <diffuse>0.22 0.22 0.22 1</diffuse>
-      <specular>0.10 0.10 0.10 1</specular>
-    </material>
+    <material>Gazebo/DarkGrey</material>
   </gazebo>
   <!-- ═══════════════════════════════════════════════════════════════════
@@ -191,9 +167,5 @@
   </link>
   <gazebo reference="${robot_ns}/lidar_housing_link">
-    <material>
-      <ambient>0.10 0.10 0.10 1</ambient>
-      <diffuse>0.12 0.12 0.12 1</diffuse>
-      <specular>0.08 0.08 0.08 1</specular>
-    </material>
+    <material>Gazebo/Black</material>
   </gazebo>
   <!-- ═══════════════════════════════════════════════════════════════════
